File: leaf_type_00/leaf_type_00.brd (EAGLE design)
At the start: 28 x 13 mm, 2 parts, among them J1 CONN_5X2_1P00_IN, J2 TC_2050_IDC_NL_TOP

Commit message: working on leafs
Parts:
- removed J2: TC_2050_IDC_NL_TOP, leaf:TC_2050_IDC_NL_TOP
- added C1, C2: (no value), stepOSP:0805
- added J5, J6: CONN_04_JST_PA, leaf:CONN_04_JST_PA
- added U$1: TPS709XX, stepOSP:SOT23-5
- added U$2: BMA280, stepOSP:BMA280
- added U$3, U$4: RS422_TRANSCEIVER_ISL83488, stepOSP:SO-08
- added U$5: BMI-S-103, stepOSP:BMI-S-103
- added U1: STM32F103RBT6, leaf:STM32_TQFP_64_10X10
- J1: value CONN_5X2_1P00_IN -> TC_2050_IDC_NL_TOP; device leaf:CONN_5X2_0P100_IN -> leaf:TC_2050_IDC_NL_TOP
- moved J1 16.1 mm to (33.0, 2.54), turned to 180 degrees
Connections:
- removed net 1: J1.1, J2.1
- removed net 10: J1.2, J2.10
- removed net 2: J1.3, J2.2
- removed net 3: J1.5, J2.3
- removed net 4: J1.7, J2.4
- removed net 5: J1.9, J2.5
- removed net 6: J1.10, J2.6
- removed net 7: J1.8, J2.7
- removed net 8: J1.6, J2.8
- removed net 9: J1.4, J2.9
Routing:
- net 5: track 10.2 -> 0.00 mm
- net 6: track 9.52 -> 0.00 mm, vias 1 -> 0
- net 10: track 9.30 -> 0.00 mm, vias 1 -> 0
- net 7: track 8.83 -> 0.00 mm, vias 1 -> 0
- net 9: track 8.75 -> 0.00 mm, vias 1 -> 0
- net 4: track 8.58 -> 0.00 mm
- net 8: track 8.26 -> 0.00 mm, vias 1 -> 0
- net 3: track 8.18 -> 0.00 mm
- net 1: track 8.12 -> 0.00 mm
- net 2: track 7.58 -> 0.00 mm
Other:
- board size 28 x 13 mm -> 49.6 x 36 mm
- board text removed: "Project Leaf"
